File: PWD665.kicad_pcb (KiCad board)
At the start: 2 copper layers, 380 x 237.5 mm, 21 parts, among them IC21 uPD4990AC, IC65 D65101GD110, X2 32.768K

Commit message: add CN2 FDD connector
Parts:
- added C66: C_Small, Capacitor_SMD:C_1206_3216Metric, B.Cu at (171.2, 44.4)
- added CN2: FDD, 88va_Library:HRS_HIF6-68PA, F.Cu at (140.9, 211.1)
- added CN5: LED, Connector_JST:JST_EH_B4B-EH-A_1x04_P2.50mm_Vertical, F.Cu at (17.7, 50.5)
- added IC20: 7407, Package_DIP:DIP-14_W7.62mm, F.Cu at (167.6, 48.2)
- added LC23: Filter_EMI_LCL, 88va_Library:Filter, F.Cu at (17.7, 70.2)
- added LC6: Filter_EMI_LCL, 88va_Library:Filter, F.Cu at (20.3, 39.7)
- added LC7: Filter_EMI_LCL, 88va_Library:Filter, F.Cu at (36.1, 27.6)
- added LC8: Filter_EMI_LCL, 88va_Library:Filter, F.Cu at (46.0, 27.6)
Connections:
- IC65 pad 1: +5V -> unconnected-(IC65-VDD-Pad1)
- IC65 pad 145: (no net) -> Net-(IC65-_?)
- IC65 pad 40: +5V -> unconnected-(IC65-VDD-Pad40)
- IC65 pad 51: (no net) -> Net-(IC65-_STP)
- IC65 pad 65: (no net) -> Net-(IC65-_LEDVa)
- IC65 pad 66: (no net) -> Net-(IC65-_LEDVb)
- IC65 pad 67: (no net) -> Net-(IC65-_LEDVc)
- IC65 pad 71: CDI -> unconnected-(IC65-CLDI-Pad71)
- IC65 pad 74: C2 -> unconnected-(IC65-CLC2-Pad74)
- IC65 pad 75: C1 -> unconnected-(IC65-CLC1-Pad75)
- IC65 pad 76: C0 -> unconnected-(IC65-CLC0-Pad76)
- IC65 pad 77: CSTB -> unconnected-(IC65-CLSTB-Pad77)
- IC65 pad 78: CDO -> unconnected-(IC65-CLDO-Pad78)
- IC65 pad 82: CCLK -> unconnected-(IC65-CLCLK-Pad82)
Routing:
- net unconnected-(IC65-CLDI-Pad71): track 0.00 -> 18.1 mm, vias 0 -> 2
- net CDI: track 289.6 -> 271.5 mm, vias 3 -> 1
Other:
- board text added: "A1"
- board text added: "B1"

Commit message: add CN4 TEXT BUS
Parts:
- added CN4: TEXT BUS, 88va_Library:FCI_PI96B30RD-6TR2, F.Cu at (219.0, 63.2)
- added IC22: DIP-14_W7.62mm, Package_DIP:DIP-14_W7.62mm, F.Cu at (192.7, 66.3)
- moved LC7 0.63 mm to (36.1, 28.2)
- moved LC8 0.63 mm to (46.0, 28.2)
- moved MR10 0.32 mm to (192.7, 56.2)
- moved MR9 0.32 mm to (192.7, 51.1)
- turned C66 to 0 degrees
Connections:
- C66 pad 1: unconnected-(C66-Pad1) -> +5V
- IC20 pad 8: CN4_C25 -> XARESET?
- IC65 pad 71: unconnected-(IC65-CLDI-Pad71) -> CDI
- LC23 pad 1: unconnected-(LC23-Pad1) -> +5V
Routing:
- net Net-(IC65-_LEDVc): track 0.00 -> 472.1 mm, vias 0 -> 1
- net Net-(IC65-_LEDVb): track 0.00 -> 467.7 mm, vias 0 -> 1
- net Net-(IC65-_LEDVa): track 0.00 -> 463.9 mm, vias 0 -> 1
- net Net-(IC65-XARESET?): track 0.00 -> 303.2 mm, vias 0 -> 4
- net Net-(IC20-Pad2): track 0.00 -> 190.2 mm, vias 0 -> 1
- net Net-(IC20-Pad4): track 0.00 -> 164.4 mm
- net Net-(IC20-Pad6): track 0.00 -> 159.6 mm
- net XARESET?: track 0.00 -> 126.7 mm, vias 0 -> 4
- net GND: track 50.4 -> 139.7 mm, vias 3 -> 4
- net MSWCS: track 41.0 -> 121.0 mm, vias 1 -> 3
- net BACKUP: track 100.9 -> 180.3 mm, vias 2 -> 4
- net Net-(CN5-Pin_2): track 0.00 -> 65.2 mm
- net Net-(CN5-Pin_3): track 0.00 -> 59.7 mm
- net (no net): track 1682.1 -> 1731.3 mm, vias 4 -> 29
- net Net-(IC65-_STP): track 0.00 -> 47.9 mm, vias 0 -> 1
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- added copper zone on F.Cu, net (none)
Other:
- board text added: "C104"
- board text added: "C74"
- board text added: "C84"
- board text added: "IC16ソケットの下へ"
- board text added: "IC31とIC43の合間"
- board text added: "R63"
