File: calendar_battery.kicad_sch (KiCad schematic)
At the start: 20 parts, among them IC21 uPD4990AC, Q10 Q_PNP, Q11 Q_PNP, Q9 Q_NPN, X2 32.768K

Commit message: schematic: tidy hierarchical sheets
Other:
- title: (none) -> カレンダクロック・バックアップ電池
Changed lines of the file:
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@@
 (kicad_sch (version 20230121) (generator eeschema)
   (paper "A4")
+  (title_block
+    (title "カレンダクロック・バックアップ電池")
+    (comment 1 "VA1回路図 P.262")
+  )
   (junction (at 72.39 120.65) (diameter 0) (color 0 0 0 0)
   )
