File: fdd.kicad_sch (KiCad schematic)
At the start: 1 part, among them CN2 FDD

Commit message: schematic: tidy hierarchical sheets
Other:
- title: (none) -> FDDコネクタ
Changed lines of the file:
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@@
 (kicad_sch (version 20230121) (generator eeschema)
   (paper "A4")
+  (title_block
+    (title "FDDコネクタ")
+    (comment 1 "VA1回路図 P.245")
+  )
   (junction (at 116.84 139.7) (diameter 0) (color 0 0 0 0)
   )
